File: pcb/DeskHop.kicad_sch (KiCad schematic)
At the start: 12 parts, among them J1 Keyboard In, J2 Debug2, J3 Debug1, J4 Mouse In, U1 Pico Primary, U2 Pico Secondary, U4 ADuM1201BR

Commit message: Add switch to PCB board
Parts:
- added SW1, SW2: SW_Push, Button_Switch_THT:SW_PUSH_1P1T_6x3.5mm_H5.0_APEM_MJTP1250, symbol Switch:SW_Push
Connections:
- net GND: now also SW2.1
- net GND2: now also SW1.1
- net at U1.14 (GPIO10): now also SW1.2
- net at U2.14 (GPIO10): now also SW2.2
Changed lines of the file:
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@@
   (junction (at 88.9 135.89) (diameter 0) (color 0 0 0 0)
   )
+  (junction (at 175.26 87.63) (diameter 0) (color 0 0 0 0)
+  )
   (junction (at 74.93 93.98) (diameter 0) (color 0 0 0 0)
   )
@@
   (junction (at 175.26 57.15) (diameter 0) (color 0 0 0 0)
   )
+  (junction (at 48.26 88.9) (diameter 0) (color 0 0 0 0)
+  )
   (junction (at 190.5 69.85) (diameter 0) (color 0 0 0 0)
   )
@@
   (junction (at 190.5 130.81) (diameter 0) (color 0 0 0 0)
   )
-  (junction (at 71.12 83.82) (diameter 0) (color 0 0 0 0)
-  )
   (junction (at 212.09 109.22) (diameter 0) (color 0 0 0 0)
   )
@@
     (stroke (width 0) (type default))
   )
+  (wire (pts (xy 48.26 88.9) (xy 48.26 92.71))
+    (stroke (width 0) (type default))
+  )
+  (wire (pts (xy 186.69 85.09) (xy 186.69 87.63))
+    (stroke (width 0) (type default))
+  )
   (wire (pts (xy 71.12 99.06) (xy 71.12 121.92))
     (stroke (width 0) (type default))
@@
     (stroke (width 0) (type default))
   )
+  (wire (pts (xy 48.26 71.12) (xy 71.12 71.12))
+    (stroke (width 0) (type default))
+  )
+  (wire (pts (xy 48.26 88.9) (xy 57.15 88.9))
+    (stroke (width 0) (type default))
+  )
+  (wire (pts (xy 185.42 87.63) (xy 186.69 87.63))
+    (stroke (width 0) (type default))
+  )
   (wire (pts (xy 198.12 132.08) (xy 198.12 135.89))
     (stroke (width 0) (type default))
@@
     (stroke (width 0) (type default))
   )
+  (wire (pts (xy 48.26 71.12) (xy 48.26 88.9))
+    (stroke (width 0) (type default))
+  )
   (wire (pts (xy 71.12 71.12) (xy 71.12 58.42))
     (stroke (width 0) (type default))
@@
     (stroke (width 0) (type default))
   )
+  (wire (pts (xy 175.26 73.66) (xy 175.26 87.63))
+    (stroke (width 0) (type default))
+  )
   (wire (pts (xy 81.28 132.08) (xy 81.28 139.7))
     (stroke (width 0) (type default))
@@
     (stroke (width 0) (type default))
   )
-  (wire (pts (xy 175.26 73.66) (xy 175.26 95.25))
-    (stroke (width 0) (type default))
-  )
   (wire (pts (xy 190.5 130.81) (xy 190.5 135.89))
     (stroke (width 0) (type default))
@@
     (stroke (width 0) (type default))
   )
+  (wire (pts (xy 186.69 85.09) (xy 194.31 85.09))
+    (stroke (width 0) (type default))
+  )
   (wire (pts (xy 143.51 66.04) (xy 144.78 66.04))
     (stroke (width 0) (type default))
@@
     (stroke (width 0) (type default))
   )
+  (wire (pts (xy 74.93 88.9) (xy 77.47 88.9))
+    (stroke (width 0) (type default))
+  )
   (wire (pts (xy 175.26 118.11) (xy 175.26 120.65))
     (stroke (width 0) (type default))
@@
     (stroke (width 0) (type default))
   )
+  (wire (pts (xy 67.31 86.36) (xy 67.31 88.9))
+    (stroke (width 0) (type default))
+  )
   (wire (pts (xy 110.49 53.34) (xy 114.3 53.34))
     (stroke (width 0) (type default))
@@
     (stroke (width 0) (type default))
   )
+  (wire (pts (xy 67.31 86.36) (xy 74.93 86.36))
+    (stroke (width 0) (type default))
+  )
   (wire (pts (xy 190.5 57.15) (xy 190.5 69.85))
     (stroke (width 0) (type default))
@@
   )
   (wire (pts (xy 58.42 96.52) (xy 58.42 105.41))
+    (stroke (width 0) (type default))
+  )
+  (wire (pts (xy 175.26 87.63) (xy 175.26 95.25))
     (stroke (width 0) (type default))
   )
@@
     )
   )
-  (symbol (lib_id "power:GND2") (at 71.12 83.82 0) (mirror y) (unit 1)
+  (symbol (lib_id "power:GND2") (at 48.26 92.71 0) (mirror y) (unit 1)
     (in_bom yes) (on_board yes) (dnp no)
-    (property "Reference" "#PWR07" (at 71.12 90.17 0)
-      (effects (font (size 1.27 1.27)) hide)
-    )
-    (property "Value" "GND2" (at 71.12 88.9 0)
-      (effects (font (size 1.27 1.27)))
-    )
-    (property "Footprint" "" (at 71.12 83.82 0)
-      (effects (font (size 1.27 1.27)) hide)
-    )
-    (property "Datasheet" "" (at 71.12 83.82 0)
+    (property "Reference" "#PWR07" (at 48.26 99.06 0)
+      (effects (font (size 1.27 1.27)) hide)
+    )
+    (property "Value" "GND2" (at 48.26 97.79 0)
+      (effects (font (size 1.27 1.27)))
+    )
+    (property "Footprint" "" (at 48.26 92.71 0)
+      (effects (font (size 1.27 1.27)) hide)
+    )
+    (property "Datasheet" "" (at 48.26 92.71 0)
       (effects (font (size 1.27 1.27)) hide)
     )
@@
         (path "/fa1c3e0e-91b1-4532-8b22-6d396d71c75b"
           (reference "H2") (unit 1)
+        )
+      )
+    )
+  )
+  (symbol (lib_id "Switch:SW_Push") (at 62.23 88.9 0) (unit 1)
+    (in_bom yes) (on_board yes) (dnp no) (fields_autoplaced)
+    (property "Reference" "SW1" (at 62.23 81.28 0)
+      (effects (font (size 1.27 1.27)))
+    )
+    (property "Value" "SW_Push" (at 62.23 83.82 0)
+      (effects (font (size 1.27 1.27)))
+    )
+    (property "Footprint" "Button_Switch_THT:SW_PUSH_1P1T_6x3.5mm_H5.0_APEM_MJTP1250" (at 62.23 83.82 0)
+      (effects (font (size 1.27 1.27)) hide)
+    )
+    (property "Datasheet" "~" (at 62.23 83.82 0)
+      (effects (font (size 1.27 1.27)) hide)
+    )
+    (pin "1")
+    (pin "2")
+    (instances
+      (project "DeskHop"
+        (path "/fa1c3e0e-91b1-4532-8b22-6d396d71c75b"
+          (reference "SW1") (unit 1)
         )
       )
@@
         )
       )
+    )
+  )
+  (symbol (lib_id "Switch:SW_Push") (at 180.34 87.63 0) (unit 1)
+    (in_bom yes) (on_board yes) (dnp no) (fields_autoplaced)
+    (property "Reference" "SW2" (at 180.34 80.01 0)
+      (effects (font (size 1.27 1.27)))
+    )
+    (property "Value" "SW_Push" (at 180.34 82.55 0)
+      (effects (font (size 1.27 1.27)))
+    )
+    (property "Footprint" "Button_Switch_THT:SW_PUSH_1P1T_6x3.5mm_H5.0_APEM_MJTP1250" (at 180.34 82.55 0)
+      (effects (font (size 1.27 1.27)) hide)
+    )
+    (property "Datasheet" "~" (at 180.34 82.55 0)
+      (effects (font (size 1.27 1.27)) hide)
+    )
+    (pin "1")
+    (pin "2")
+    (instances
+      (project "DeskHop"
+        (path "/fa1c3e0e-91b1-4532-8b22-6d396d71c75b"
+          (reference "SW2") (unit 1)
+        )
+      )
